Commit message: cleaned up

File: conf/au_crustcrawler_ax12.urdf (robot description, URDF)
Before this commit: robot test_robot, 6 links, 5 joints
Links:
- removed link base_arm
- removed link gripper_link
- added link base_arm_1; visual box size=0.03 0.1 0.03
- added link base_arm_2; visual box size=0.08 0.03 0.11
- added link gripper_camera_plate; visual box size=0.05 0.06 0.005
- added link gripper_end_effector; visual box size=0.03 0.03 0.15
- added link gripper_servo_base; visual box size=0.045 0.03 0.03
- added link wrist_temp; visual box size=0.03 0.045 0.03
Joints:
- removed joint gripper_linkage
- added joint gripper_linkage_cameraplate: type fixed, parent wrist, child gripper_camera_plate, origin xyz=0 0.0 0.001 rpy=0 0 0
- added joint gripper_linkage_end_effector: type fixed, parent gripper_servo_base, child gripper_end_effector, origin xyz=0.025 0.015 0.15 rpy=0 0 0
- added joint gripper_linkage_servo: type fixed, parent gripper_camera_plate, child gripper_servo_base, origin xyz=-0.025 -0.015 0.025 rpy=0 0 0
- added joint linkage: type fixed, parent base_arm_1, child base_arm_2, origin xyz=0 0 0.03 rpy=1.5707 -0.707 0, axis 0 0 1
- added joint wrist_linkage: type fixed, parent middle_arm, child wrist_temp, origin xyz=0.03 0.0 0 rpy=3.1415 0 0
- joint joint1: child base_arm -> base_arm_1; limit lower=-1.5 upper=1.5 effort=1000.0 velocity=1.0 -> lower=-1.3 upper=1.3 effort=1000.0 velocity=1.0
- joint joint2: limit lower=-1.3 upper=2.2 effort=1000.0 velocity=1.0 -> lower=-1.9 upper=2.2 effort=1000.0 velocity=1.0; origin xyz=0.08 0 0.1 rpy=1.5707 -0.785398163 0 -> xyz=0.08 0 0 rpy=0 0 0; parent base_arm -> base_arm_2
- joint joint3: origin xyz=0.17 0 0 rpy=3.1415 0 1.5707 -> xyz=0.17 0 0 rpy=3.1415 0 0
- joint joint4: limit lower=-1.4 upper=1.4 effort=1000.0 velocity=1.0 -> lower=-2.2 upper=2.2 effort=1000.0 velocity=1.0; parent middle_arm -> wrist_temp

Commit message: Updated urdf to new robot configuration

File: conf/au_crustcrawler_ax12.urdf (robot description, URDF)
Before this commit: robot test_robot, 10 links, 9 joints
Links:
- removed link base_arm_1
- removed link base_arm_2
- added link base_arm; visual box size=0.03 0.03 0.18
Joints:
- removed joint linkage
- joint joint1: child base_arm_1 -> base_arm
- joint joint2: origin xyz=0.08 0 0 rpy=0 0 0 -> xyz=0 0 0.15 rpy=1.5707 -1.5707 0; parent base_arm_2 -> base_arm
- joint joint3: origin xyz=0.17 0 0 rpy=3.1415 0 0 -> xyz=0.17 0 0 rpy=0 0 0
- joint wrist_linkage: origin xyz=0.03 0.0 0 rpy=3.1415 0 0 -> xyz=0.03 0.0 0 rpy=0 0 0

Commit message: updated meta to ignore gripper joint

File: conf/au_crustcrawler_ax12.urdf (robot description, URDF)
Before this commit: robot test_robot, 9 links, 8 joints
Joints:
- joint joint1: limit lower=-1.3 upper=1.3 effort=1000.0 velocity=1.0 -> lower=-1.3 upper=1.3 effort=1000.0 velocity=0.2
- joint joint2: limit lower=-1.9 upper=2.2 effort=1000.0 velocity=1.0 -> lower=-2.48 upper=2.48 effort=1000.0 velocity=0.2
- joint joint3: limit lower=-1.3 upper=2.2 effort=1000.0 velocity=1.0 -> lower=-2.48 upper=2.48 effort=1000.0 velocity=0.2
- joint joint4: limit lower=-2.2 upper=2.2 effort=1000.0 velocity=1.0 -> lower=-2.48 upper=2.48 effort=1000.0 velocity=0.2

Commit message: Increased joint range

File: conf/au_crustcrawler_ax12.urdf (robot description, URDF)
Before this commit: robot test_robot, 9 links, 8 joints
Joints:
- joint joint1: limit lower=-1.3 upper=1.3 effort=1000.0 velocity=0.2 -> lower=-2.48 upper=2.48 effort=1000.0 velocity=0.2

Commit message: Updated base to include inverse kinematics for the crustcrawler - untested on real robot

File: conf/au_crustcrawler_ax12.urdf (robot description, URDF)
Before this commit: robot test_robot, 9 links, 8 joints
Links:
- removed link gripper_camera_plate
- removed link gripper_servo_base
- removed link wrist
- removed link wrist_temp
- link gripper_end_effector: geometry visual box size=0.03 0.03 0.2
Joints:
- removed joint gripper_linkage_cameraplate
- removed joint gripper_linkage_end_effector
- removed joint gripper_linkage_servo
- removed joint wrist_linkage
- joint joint1: origin xyz= 0 0 0.04 rpy=0 0 0 -> xyz= 0 0 0.00 rpy=0 0 0
- joint joint2: origin xyz=0 0 0.15 rpy=1.5707 -1.5707 0 -> xyz=0 0 0.1 rpy=0 -1.57 -1.57 
- joint joint3: origin xyz=0.17 0 0 rpy=0 0 0 -> xyz=0.20 0 0 rpy=3.145 0 0
- joint joint4: child wrist -> gripper_end_effector; origin xyz=0.035 0.025 0 rpy=0 1.5707 0 -> xyz=0.2 0.0 0.0 rpy=0 1.5707 0; parent wrist_temp -> middle_arm

Commit message: Update au_crustcrawler_ax12.urdf
joint3 rpy "3.145 0 0" -> "0 0 0", for correct visualization in rviz of joint 3

File: conf/au_crustcrawler_ax12.urdf (robot description, URDF)
Before this commit: robot test_robot, 5 links, 4 joints
Joints:
- joint joint3: origin xyz=0.20 0 0 rpy=3.145 0 0 -> xyz=0.20 0 0 rpy=0 0 0
